File: MechKeyboard1/MechKeyboard1.sch (KiCad schematic (older format))
At the start: 21 parts, among them J1 AVR-ISP-6, SW1 SW_SKQG, U1 ATmega32U4-AU, U2 PRTR5V0U2X, X1 XTAL

Commit message: Schematic Done! Pre-FootPrint
*De-Bug Schematic
*Tidy up Custom Symbol
Parts:
- R1: value R_Small -> 10k
- SW1: value SW_SKQG -> SW_Push_Reset
Connections:
- net +5V: now also U1.7 (VBUS)
- net D+: now also U1.4 (D+)
- net D-: now also U1.3 (D-)
- net RESET: now also U1.13 (~RESET)
- net row0: now reaches U1.1 (PE6)
- net col8: now reaches U1.19 (PD1)
- net col9: now reaches U1.20 (PD2)
- net col10: now reaches U1.21 (PD3)
- net col12: now reaches U1.22 (PD5)
- net col11: now reaches U1.25 (PD4)
- net col13: now reaches U1.26 (PD6)
- net col14: now reaches U1.27 (PD7)
- net col0: now reaches U1.28 (PB4)
- net col1: now reaches U1.29 (PB5)
- net col2: now reaches U1.30 (PB6)
- net col3: now reaches U1.31 (PC6)
- net col4: now reaches U1.32 (PC7)
- net col6: now reaches U1.36 (PF7)
- net col5: now reaches U1.37 (PF6)
- net row1: now reaches U1.38 (PF5)
- net row4: now reaches U1.39 (PF4)
- net row3: now reaches U1.40 (PF1)
- net row2: now reaches U1.41 (PF0)
- net col7: now reaches U1.8 (PB0)
- no-connect marks 4 -> 7
Other:
- moved on the sheet: R2
Changed lines of the file:
@@
 	1    0    0    -1
 $EndComp
-Wire Wire Line
-	3250 5350 3150 5350
-$Comp
-L power:GND #PWR013
+$Comp
+L power:GND #PWR014
 U 1 1 60704592
 P 2700 5500
-F 0 "#PWR013" H 2700 5250 50  0001 C CNN
+F 0 "#PWR014" H 2700 5250 50  0001 C CNN
 F 1 "GND" H 2705 5327 50  0000 C CNN
 F 2 "" H 2700 5500 50  0001 C CNN
@@
 	1    0    0    -1
 $EndComp
-Wire Wire Line
-	3150 5350 2700 5350
-Wire Wire Line
-	2700 5350 2700 5500
-Connection ~ 3150 5350
 Text GLabel 2550 2250 0    50   Input ~ 0
 XTAL1
@@
 Wire Wire Line
 	2550 2450 2650 2450
-Wire Wire Line
-	3850 4150 4200 4150
-$Comp
-L Device:R_Small R2
-U 1 1 60707147
-P 4300 4150
-F 0 "R2" V 4104 4150 50  0000 C CNN
-F 1 "10k" V 4195 4150 50  0000 C CNN
-F 2 "" H 4300 4150 50  0001 C CNN
-F 3 "~" H 4300 4150 50  0001 C CNN
-	1    4300 4150
-	0    1    1    0
-$EndComp
-$Comp
-L power:GND #PWR010
+$Comp
+L power:GND #PWR011
 U 1 1 60708810
-P 4750 4300
-F 0 "#PWR010" H 4750 4050 50  0001 C CNN
-F 1 "GND" H 4755 4127 50  0000 C CNN
-F 2 "" H 4750 4300 50  0001 C CNN
-F 3 "" H 4750 4300 50  0001 C CNN
-	1    4750 4300
-	1    0    0    -1
-$EndComp
-Wire Wire Line
-	4400 4150 4750 4150
-Wire Wire Line
-	4750 4150 4750 4300
-NoConn ~ 3850 4250
+P 4750 4400
+F 0 "#PWR011" H 4750 4150 50  0001 C CNN
+F 1 "GND" H 4755 4227 50  0000 C CNN
+F 2 "" H 4750 4400 50  0001 C CNN
+F 3 "" H 4750 4400 50  0001 C CNN
+	1    4750 4400
+	1    0    0    -1
+$EndComp
 $Comp
 L Device:C_Small C8
@@
 $EndComp
 $Comp
-L power:GND #PWR09
+L power:GND #PWR010
 U 1 1 6070A5CB
-P 2400 3850
-F 0 "#PWR09" H 2400 3600 50  0001 C CNN
-F 1 "GND" H 2405 3677 50  0000 C CNN
-F 2 "" H 2400 3850 50  0001 C CNN
-F 3 "" H 2400 3850 50  0001 C CNN
-	1    2400 3850
-	1    0    0    -1
-$EndComp
-Wire Wire Line
-	2650 3350 2400 3350
-Wire Wire Line
-	2400 3350 2400 3400
-Wire Wire Line
-	2400 3600 2400 3850
+P 2400 3600
+F 0 "#PWR010" H 2400 3350 50  0001 C CNN
+F 1 "GND" H 2405 3427 50  0000 C CNN
+F 2 "" H 2400 3600 50  0001 C CNN
+F 3 "" H 2400 3600 50  0001 C CNN
+	1    2400 3600
+	1    0    0    -1
+$EndComp
 NoConn ~ 2650 2650
 $Comp
@@
 	900  2950 1300 2950
 $Comp
-L power:GND #PWR07
+L power:GND #PWR08
 U 1 1 60714C79
 P 1300 3050
-F 0 "#PWR07" H 1300 2800 50  0001 C CNN
+F 0 "#PWR08" H 1300 2800 50  0001 C CNN
 F 1 "GND" H 1305 2877 50  0000 C CNN
 F 2 "" H 1300 3050 50  0001 C CNN
@@
 Wire Wire Line
 	5350 850  5350 1000
-Text GLabel 4150 2150 2    50   Input ~ 0
+Text GLabel 4500 2150 2    50   Input ~ 0
 SCK
-Text GLabel 4150 2250 2    50   Input ~ 0
+Text GLabel 4500 2250 2    50   Input ~ 0
 MOSI
-Text GLabel 4150 2350 2    50   Input ~ 0
+Text GLabel 4500 2350 2    50   Input ~ 0
 MISO
-Wire Wire Line
-	3850 2150 4150 2150
-Wire Wire Line
-	3850 2250 4150 2250
-Wire Wire Line
-	4150 2350 3850 2350
 $Comp
 L local:SW_SKQG SW1
@@
 P 6000 3650
 F 0 "SW1" H 5950 4475 50  0000 C CNN
-F 1 "SW_SKQG" H 5950 4384 50  0000 C CNN
+F 1 "SW_Push_Reset" H 5950 4384 50  0000 C CNN
 F 2 "" H 6000 3650 50  0001 C CNN
 F 3 "" H 6000 3650 50  0001 C CNN
@@
 NoConn ~ 5350 3050
 $Comp
-L power:GND #PWR08
+L power:GND #PWR09
 U 1 1 60739FD3
 P 5100 3700
-F 0 "#PWR08" H 5100 3450 50  0001 C CNN
+F 0 "#PWR09" H 5100 3450 50  0001 C CNN
 F 1 "GND" H 5105 3527 50  0000 C CNN
 F 2 "" H 5100 3700 50  0001 C CNN
@@
 P 6950 2700
 F 0 "R1" H 7009 2746 50  0000 L CNN
-F 1 "R_Small" H 7009 2655 50  0000 L CNN
+F 1 "10k" H 7009 2655 50  0000 L CNN
 F 2 "" H 6950 2700 50  0001 C CNN
 F 3 "~" H 6950 2700 50  0001 C CNN
@@
 	6150 4500 6250 4500
 Wire Wire Line
-	6250 5700 6150 5700
+	6250 5700 6200 5700
 Wire Wire Line
 	6150 5100 6700 5100
@@
 Connection ~ 6400 4600
 $Comp
-L power:+5V #PWR012
+L power:+5V #PWR013
 U 1 1 607709B3
 P 7600 4600
-F 0 "#PWR012" H 7600 4450 50  0001 C CNN
+F 0 "#PWR013" H 7600 4450 50  0001 C CNN
 F 1 "+5V" V 7615 4728 50  0000 L CNN
 F 2 "" H 7600 4600 50  0001 C CNN
@@
 $EndComp
 $Comp
-L power:VCC #PWR011
+L power:VCC #PWR012
 U 1 1 607730C0
 P 7150 4550
-F 0 "#PWR011" H 7150 4400 50  0001 C CNN
+F 0 "#PWR012" H 7150 4400 50  0001 C CNN
 F 1 "VCC" H 7165 4723 50  0000 C CNN
 F 2 "" H 7150 4550 50  0001 C CNN
@@
 $EndComp
 Wire Wire Line
-	6400 4600 7150 4600
+	6400 4600 6700 4600
 Wire Wire Line
 	7150 4550 7150 4600
@@
 	7150 4600 7250 4600
 Wire Wire Line
-	7450 4600 7600 4600
+	7450 4600 7550 4600
 $Comp
 L Device:R_Small R5
@@
 $EndComp
 $Comp
-L power:GND #PWR015
+L power:GND #PWR016
 U 1 1 6077F342
 P 6450 6000
-F 0 "#PWR015" H 6450 5750 50  0001 C CNN
+F 0 "#PWR016" H 6450 5750 50  0001 C CNN
 F 1 "GND" H 6455 5827 50  0000 C CNN
 F 2 "" H 6450 6000 50  0001 C CNN
@@
 $EndComp
 $Comp
-L power:VCC #PWR014
+L power:VCC #PWR015
 U 1 1 6078D611
 P 7150 5850
-F 0 "#PWR014" H 7150 5700 50  0001 C CNN
+F 0 "#PWR015" H 7150 5700 50  0001 C CNN
 F 1 "VCC" V 7165 5977 50  0000 L CNN
 F 2 "" H 7150 5850 50  0001 C CNN
@@
 F1 "matrix.sch" 50
 $EndSheet
+Text GLabel 3850 2050 2    50   Input ~ 0
+col7
+Text GLabel 3850 2450 2    50   Input ~ 0
+col0
+Text GLabel 3850 2550 2    50   Input ~ 0
+col1
+Text GLabel 3850 2650 2    50   Input ~ 0
+col2
+NoConn ~ 3850 2750
+Text GLabel 3850 2950 2    50   Input ~ 0
+col3
+Text GLabel 3850 3050 2    50   Input ~ 0
+col4
+Wire Wire Line
+	3850 2150 4500 2150
+Wire Wire Line
+	3850 2250 4500 2250
+Wire Wire Line
+	3850 2350 4500 2350
+NoConn ~ 3850 3250
+Text GLabel 3850 3350 2    50   Input ~ 0
+col8
+Text GLabel 3850 3450 2    50   Input ~ 0
+col9
+Text GLabel 3850 3550 2    50   Input ~ 0
+col10
+Text GLabel 3850 3650 2    50   Input ~ 0
+col11
+Text GLabel 3850 3750 2    50   Input ~ 0
+col12
+Text GLabel 3850 3850 2    50   Input ~ 0
+col13
+Text GLabel 3850 3950 2    50   Input ~ 0
+col14
+Text GLabel 3850 4250 2    50   Input ~ 0
+row0
+Text GLabel 3850 4450 2    50   Input ~ 0
+row2
+Text GLabel 3850 4550 2    50   Input ~ 0
+row3
+Text GLabel 3850 4650 2    50   Input ~ 0
+row4
+Text GLabel 3850 4750 2    50   Input ~ 0
+row1
+Text GLabel 3850 4850 2    50   Input ~ 0
+col5
+Text GLabel 3850 4950 2    50   Input ~ 0
+col6
+Text GLabel 2650 3050 0    50   Input ~ 0
+D+
+Text GLabel 2650 3150 0    50   Input ~ 0
+D-
+$Comp
+L power:+5V #PWR07
+U 1 1 6138DFAD
+P 2650 2850
+F 0 "#PWR07" H 2650 2700 50  0001 C CNN
+F 1 "+5V" H 2665 3023 50  0000 C CNN
+F 2 "" H 2650 2850 50  0001 C CNN
+F 3 "" H 2650 2850 50  0001 C CNN
+	1    2650 2850
+	0    -1   -1   0
+$EndComp
+Text GLabel 2650 2050 0    50   Input ~ 0
+RESET
+NoConn ~ 6150 4700
+NoConn ~ 6150 5300
+$Comp
+L power:PWR_FLAG #FLG01
+U 1 1 6139D706
+P 6700 4600
+F 0 "#FLG01" H 6700 4675 50  0001 C CNN
+F 1 "PWR_FLAG" H 6700 4773 50  0000 C CNN
+F 2 "" H 6700 4600 50  0001 C CNN
+F 3 "~" H 6700 4600 50  0001 C CNN
+	1    6700 4600
+	1    0    0    -1
+$EndComp
+Connection ~ 6700 4600
+Wire Wire Line
+	6700 4600 7150 4600
+$Comp
+L power:PWR_FLAG #FLG02
+U 1 1 6139EDB4
+P 7550 4600
+F 0 "#FLG02" H 7550 4675 50  0001 C CNN
+F 1 "PWR_FLAG" H 7550 4773 50  0000 C CNN
+F 2 "" H 7550 4600 50  0001 C CNN
+F 3 "~" H 7550 4600 50  0001 C CNN
+	1    7550 4600
+	1    0    0    -1
+$EndComp
+Connection ~ 7550 4600
+Wire Wire Line
+	7550 4600 7600 4600
+Wire Wire Line
+	3850 4150 4750 4150
+$Comp
+L Device:R_Small R2
+U 1 1 60707147
+P 4750 4300
+F 0 "R2" V 4554 4300 50  0000 C CNN
+F 1 "10k" V 4645 4300 50  0000 C CNN
+F 2 "" H 4750 4300 50  0001 C CNN
+F 3 "~" H 4750 4300 50  0001 C CNN
+	1    4750 4300
+	-1   0    0    1
+$EndComp
+Wire Wire Line
+	4750 4150 4750 4200
+Wire Wire Line
+	2650 3350 2400 3350
+Wire Wire Line
+	2400 3350 2400 3400
+Wire Wire Line
+	3250 5350 3150 5350
+Wire Wire Line
+	3150 5350 2700 5350
+Wire Wire Line
+	2700 5350 2700 5500
+Connection ~ 3150 5350
+$Comp
+L power:PWR_FLAG #FLG0101
+U 1 1 613B149E
+P 6200 5700
+F 0 "#FLG0101" H 6200 5775 50  0001 C CNN
+F 1 "PWR_FLAG" H 6200 5873 50  0000 C CNN
+F 2 "" H 6200 5700 50  0001 C CNN
+F 3 "~" H 6200 5700 50  0001 C CNN
+	1    6200 5700
+	-1   0    0    1
+$EndComp
+Connection ~ 6200 5700
+Wire Wire Line
+	6200 5700 6150 5700
 $EndSCHEMATC
